File: step_down.sch (KiCad schematic (older format))
At the start: 17 parts, among them U1 L5009

Commit message: bugs gefixt. fertigungsdaten hinzugefügt
Parts:
- C1, C5: footprint (none) -> Capacitors_SMD:c_1206
- C2, C6: footprint (none) -> Capacitors_SMD:c_0805
- C3: footprint (none) -> Capacitors_SMD:c_0402
- C4: footprint (none) -> SMD_Packages:SM0805
- D1: footprint (none) -> Diodes_SMD:Diode-SMA_Standard
- L1: footprint (none) -> toni:SRR7032_Series
- R1, R2, R3, R4: footprint (none) -> SMD_Packages:SM0402
- R5: footprint (none) -> SMD_Packages:SM1206
- U1: footprint (none) -> SMD_Packages:SSOP8-9
- gnd1, in1, out1: footprint (none) -> Connect:SIL-1
Changed lines of the file:
@@
 LIBS:valves
 LIBS:step_down-cache
-EELAYER 24 0
+EELAYER 25 0
 EELAYER END
 $Descr A4 11693 8268
@@
 F 0 "C1" H 3500 3300 40  0000 L CNN
 F 1 "Cin" H 3506 3115 40  0000 L CNN
-F 2 "" H 3538 3050 30  0000 C CNN
+F 2 "Capacitors_SMD:c_1206" H 3538 3050 30  0001 C CNN
 F 3 "" H 3500 3200 60  0000 C CNN
 F 4 "1uF" H 3500 3200 60  0001 C CNN "Bauteilwert"
@@
 F 0 "C2" H 3750 3300 40  0000 L CNN
 F 1 "Cinx" H 3756 3115 40  0000 L CNN
-F 2 "" H 3788 3050 30  0000 C CNN
+F 2 "Capacitors_SMD:c_0805" H 3788 3050 30  0001 C CNN
 F 3 "" H 3750 3200 60  0000 C CNN
 F 4 "100nF" H 3750 3200 60  0001 C CNN "Bauteilwert"
@@
 F 0 "R1" V 4580 3400 40  0000 C CNN
 F 1 "Ron" V 4507 3401 40  0000 C CNN
-F 2 "" V 4430 3400 30  0000 C CNN
+F 2 "SMD_Packages:SM0402" V 4430 3400 30  0001 C CNN
 F 3 "" H 4500 3400 30  0000 C CNN
 F 4 "332k" H 4500 3400 60  0001 C CNN "Bauteilwert"
@@
 F 0 "C3" H 6050 3550 40  0000 L CNN
 F 1 "Cb" H 6056 3365 40  0000 L CNN
-F 2 "" H 6088 3300 30  0000 C CNN
+F 2 "Capacitors_SMD:c_0402" H 6088 3300 30  0001 C CNN
 F 3 "" H 6050 3450 60  0000 C CNN
 F 4 "10nF" H 6050 3450 60  0001 C CNN "Bauteilwert"
@@
 F 0 "D1" H 6400 3550 40  0000 C CNN
 F 1 "DIODESCH" H 6400 3350 40  0000 C CNN
-F 2 "" H 6400 3450 60  0000 C CNN
+F 2 "Diodes_SMD:Diode-SMA_Standard" H 6400 3450 60  0001 C CNN
 F 3 "" H 6400 3450 60  0000 C CNN
 F 4 "1A 750mV" H 6400 3450 60  0001 C CNN "Bauteilwert"
@@
 F 0 "L1" H 6750 3750 50  0000 C CNN
 F 1 "INDUCTOR_SMALL" H 6750 3600 50  0000 C CNN
-F 2 "" H 6750 3650 60  0000 C CNN
+F 2 "toni:SRR7032_Series" H 6750 3650 60  0001 C CNN
 F 3 "" H 6750 3650 60  0000 C CNN
 F 4 "470uH 1,4mOhm" H 6750 3650 60  0001 C CNN "Bauteilwert"
@@
 F 0 "R2" V 4580 3650 40  0000 C CNN
 F 1 "Rilim" V 4507 3651 40  0000 C CNN
-F 2 "" V 4430 3650 30  0000 C CNN
+F 2 "SMD_Packages:SM0402" V 4430 3650 30  0001 C CNN
 F 3 "" H 4500 3650 30  0000 C CNN
 F 4 "169k" H 4500 3650 60  0001 C CNN "Bauteilwert"
@@
 F 0 "C4" H 6150 3100 40  0000 L CNN
 F 1 "Cbyb" H 6156 2915 40  0000 L CNN
-F 2 "" H 6188 2850 30  0000 C CNN
+F 2 "SMD_Packages:SM0805" H 6188 2850 30  0001 C CNN
 F 3 "" H 6150 3000 60  0000 C CNN
 F 4 "470nF" H 6150 3000 60  0001 C CNN "Bauteilwert"
@@
 F 0 "C5" H 7200 3950 40  0000 L CNN
 F 1 "Cff" H 7206 3765 40  0000 L CNN
-F 2 "" H 7238 3700 30  0000 C CNN
+F 2 "Capacitors_SMD:c_1206" H 7238 3700 30  0001 C CNN
 F 3 "" H 7200 3850 60  0000 C CNN
 F 4 "5,6nF" H 7200 3850 60  0001 C CNN "Bauteilwert"
@@
 F 0 "R3" V 7580 3800 40  0000 C CNN
 F 1 "Rfbt" V 7507 3801 40  0000 C CNN
-F 2 "" V 7430 3800 30  0000 C CNN
+F 2 "SMD_Packages:SM0402" V 7430 3800 30  0001 C CNN
 F 3 "" H 7500 3800 30  0000 C CNN
 F 4 "4,99k" H 7500 3800 60  0001 C CNN "Bauteilwert"
@@
 F 0 "R4" V 7580 4300 40  0000 C CNN
 F 1 "Rfbb" V 7507 4301 40  0000 C CNN
-F 2 "" V 7430 4300 30  0000 C CNN
+F 2 "SMD_Packages:SM0402" V 7430 4300 30  0001 C CNN
 F 3 "" H 7500 4300 30  0000 C CNN
 F 4 "1k" H 7500 4300 60  0001 C CNN "Bauteilwert"
@@
 F 0 "C6" H 7950 3850 40  0000 L CNN
 F 1 "Cout" H 7956 3665 40  0000 L CNN
-F 2 "" H 7988 3600 30  0000 C CNN
+F 2 "Capacitors_SMD:c_0805" H 7988 3600 30  0001 C CNN
 F 3 "" H 7950 3750 60  0000 C CNN
 F 4 "4,7uF" H 7950 3750 60  0001 C CNN "Bauteilwert"
@@
 F 0 "R5" V 8030 4300 40  0000 C CNN
 F 1 "Rseries" V 7950 4300 40  0000 C CNN
-F 2 "" V 7880 4300 30  0000 C CNN
+F 2 "SMD_Packages:SM1206" V 7880 4300 30  0001 C CNN
 F 3 "" H 7950 4300 30  0000 C CNN
 F 4 "500mOhm" H 7950 4300 60  0001 C CNN "Bauteilwert"
@@
 F 0 "U1" H 5650 3000 60  0000 C CNN
 F 1 "L5009" H 5350 4600 60  0000 C CNN
-F 2 "" H 5350 3650 60  0000 C CNN
+F 2 "SMD_Packages:SSOP8-9" H 5350 3650 60  0001 C CNN
 F 3 "" H 5350 3650 60  0000 C CNN
 	1    5350 3700
@@
 F 0 "in1" H 3430 3000 40  0000 L CNN
 F 1 "CONN_1" H 3350 3055 30  0001 C CNN
-F 2 "" H 3350 3000 60  0000 C CNN
+F 2 "Connect:SIL-1" H 3350 3000 60  0001 C CNN
 F 3 "" H 3350 3000 60  0000 C CNN
 	1    3350 3000
@@
 F 0 "gnd1" H 3430 3400 40  0000 L CNN
 F 1 "CONN_1" H 3350 3455 30  0001 C CNN
-F 2 "" H 3350 3400 60  0000 C CNN
+F 2 "Connect:SIL-1" H 3350 3400 60  0001 C CNN
 F 3 "" H 3350 3400 60  0000 C CNN
 	1    3350 3400
@@
 F 0 "out1" H 8180 3550 40  0000 L CNN
 F 1 "CONN_1" H 8100 3605 30  0001 C CNN
-F 2 "" H 8100 3550 60  0000 C CNN
+F 2 "Connect:SIL-1" H 8100 3550 60  0001 C CNN
 F 3 "" H 8100 3550 60  0000 C CNN
 	1    8100 3550
